File: hardware/main-board/main-board.kicad_pcb (KiCad board)
At the start: 2 copper layers, 140 x 100 mm, 61 parts, among them J1 Barrel_Jack_Switch, J10 Conn_01x04, J11 Conn_01x04, J12 Conn_01x04, J13 USB_A, J14 USB_A, J15 USB_B, J16 USB_B, J17 USB_A, J18 USB_A, J19 USB_B, J2 Conn_02x05_Odd_Even, J20 USB_B, J3 Conn_02x05_Odd_Even, J4 Conn_01x06, J5 Conn_02x05_Odd_Even, J6 Conn_02x05_Odd_Even, J7 Conn_01x05, Q1 KSP43BU, Q2 KSP43BU, Q3 KSP43BU, Q4 KSP43BU, Q5 KSP43BU, Q6 KSP43BU, Q7 KSP43BU, Q8 KSP43BU, U1 LM317_TO-220, U2 R-78E5.0-0.5, U3 LF33_TO220, U4 Omron_G3VM-41AY1, U5 Omron_G3VM-61A1, U6 Omron_G3VM-61A1, U7 Teensy4.1, U8 Omron_G3VM-61A1, U9 Omron_G3VM-61A1

Commit message: Rev A mainboard PCB
Altered to split IR relay off into isolated section
Parts:
- removed J13, J14, J17, J18: USB_A, Connector_USB:USB_A_ASSMANN_A-USB-E-R
- removed J15, J16, J19, J20: USB_B, Connector_USB:USB_B_ASSMANN_A-USBSB
- removed Q5, Q6, Q7, Q8: KSP43BU, Package_TO_SOT_THT:TO-92_Inline
- removed R17: 4.7K, Resistor_THT:R_Axial_DIN0207_L6.3mm_D2.5mm_P10.16mm_Horizontal
- removed R18, R19: 330R, Resistor_THT:R_Axial_DIN0207_L6.3mm_D2.5mm_P10.16mm_Horizontal
- removed the U5 at (188.0, 85.1)
- removed U9: Omron_G3VM-61A1, Package_DIP:DIP-4_W7.62mm
- added C7: 33pF, Capacitor_THT:C_Disc_D4.7mm_W2.5mm_P5.00mm, F.Cu at (104.1, 57.1)
- added C8: 33pF, Capacitor_THT:C_Disc_D4.7mm_W2.5mm_P5.00mm, F.Cu at (104.1, 38.1)
- added H1: MountingHole, MountingHole:MountingHole_4.3mm_M4, F.Cu at (151.1, 20.3)
- added H2: MountingHole, MountingHole:MountingHole_4.3mm_M4, F.Cu at (151.1, 108.0)
- added H3: MountingHole, MountingHole:MountingHole_4.3mm_M4, F.Cu at (24.1, 108.0)
- added H4: MountingHole, MountingHole:MountingHole_4.3mm_M4, F.Cu at (24.1, 20.3)
- added JP1: Jumper_2_Open, Jumper:SolderJumper-2_P1.3mm_Open_TrianglePad1.0x1.5mm, F.Cu at (53.3, 84.1)
- added U4: Omron_G3VM-41AY1, Package_DIP:DIP-4_W7.62mm, F.Cu at (113.0, 106.7)
- C2, C4: footprint Capacitor_SMD:C_0805_2012Metric_Pad1.18x1.45mm_HandSolder -> Capacitor_SMD:C_1210_3225Metric_Pad1.33x2.70mm_HandSolder
- J4: value Conn_01x06 -> Conn_01x04; footprint Connector_PinHeader_2.54mm:PinHeader_1x06_P2.54mm_Vertical -> Connector_PinHeader_2.54mm:PinHeader_1x04_P2.54mm_Vertical
- R12: value 4.7K -> 1.2K
- R13: value 4.7K -> 3.9K
- R14: value 330R -> 3.3K
- R15: value 330R -> 3.9K
- R16: value 4.7K -> 3.3K
- U6: value Omron_G3VM-61A1 -> MCP23016_SS; footprint Package_DIP:DIP-4_W7.62mm -> Package_DIP:DIP-28_W7.62mm
- U7: value Teensy4.1 -> MCP23016_SS; footprint Package_DIP:DIP-48_W15.24mm -> Package_DIP:DIP-28_W7.62mm
- U8: value Omron_G3VM-61A1 -> ESP32-PoE-ISO; footprint Package_DIP:DIP-4_W7.62mm -> Module:Olimex_ESP32_PoE_ISO
- moved U6 163.1 mm to (86.4, 34.3), turned to 90 degrees
- moved R13 149.0 mm to (106.7, 57.1)
- moved U8 147.8 mm to (54.6, 87.6), turned to 90 degrees
- moved R15 140.8 mm to (106.7, 38.1)
- moved R16 137.9 mm to (67.3, 57.1)
- moved R14 113.1 mm to (64.8, 57.1), turned to 180 degrees
- moved R7 111.6 mm to (65.0, 48.8)
- moved R9 106.2 mm to (119.4, 23.5), turned to 180 degrees
- moved R5 101.6 mm to (54.6, 52.1)
- moved Q3 96.9 mm to (48.9, 51.8)
- moved R4 96.5 mm to (128.3, 29.8), turned to -90 degrees
- moved R8 96.3 mm to (128.5, 55.6), turned to 90 degrees
- moved Q2 95.4 mm to (128.3, 26.7), turned to 90 degrees
- moved R3 95.2 mm to (125.2, 55.6)
- moved J9 93.6 mm to (138.4, 26.0)
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- renumbered J12 to J10, J10 to J8, J11 to J9, R5 to R10, R6 to R11, R9 to R5, R7 to R6, R8 to R7, R10 to R8, R11 to R9, U4 to U5
Connections:
- J10 pad 2: /IR_RLY_IN -> Net-(J10-Pad2)
- J2 pad 10: /P1_SW_1 -> /P4_SW_1
- J2 pad 2: /P1_LED_A -> /P4_LED_A
- J2 pad 4: /P1_LED_B -> /P4_LED_B
- J2 pad 6: /P1_LED_C -> /P4_LED_C
- J2 pad 8: /P1_SW_0 -> /P4_SW_0
- J2 pad 9: /P1_SW_2 -> /P4_SW_2
- J3 pad 10: /P2_SW_1 -> /P3_SW_1
- J3 pad 2: /P2_LED_A -> /P3_LED_A
- J3 pad 4: /P2_LED_B -> /P3_LED_B
- J3 pad 6: /P2_LED_C -> /P3_LED_C
- J3 pad 8: /P2_SW_0 -> /P3_SW_0
- J3 pad 9: /P2_SW_2 -> /P3_SW_2
- J4 pad 1: /RS232_RX -> +3V3
- J4 pad 2: /RS232_TX -> GND
- J4 pad 3: unconnected-(J4-Pad3) -> /USB_EN_A
- J4 pad 4: unconnected-(J4-Pad4) -> /USB_EN_B
- J5 pad 10: /P3_SW_1 -> /P2_SW_1
- J5 pad 2: /P3_LED_A -> /P2_LED_A
- J5 pad 4: /P3_LED_B -> /P2_LED_B
- J5 pad 6: /P3_LED_C -> /P2_LED_C
- J5 pad 8: /P3_SW_0 -> /P2_SW_0
- J5 pad 9: /P3_SW_2 -> /P2_SW_2
- J6 pad 10: /P4_SW_1 -> /P1_SW_1
- J6 pad 2: /P4_LED_A -> /P1_LED_A
- J6 pad 4: /P4_LED_B -> /P1_LED_B
- J6 pad 6: /P4_LED_C -> /P1_LED_C
- J6 pad 8: /P4_SW_0 -> /P1_SW_0
- J6 pad 9: /P4_SW_2 -> /P1_SW_2
- J7 pad 3: GND -> +5V
- R12 pad 2: /USB_EN_A -> +12VA
- R13 pad 1: Net-(Q6-Pad2) -> Net-(C7-Pad1)
- R13 pad 2: /USB_EN_B -> +3V3
- R14 pad 1: +3V3 -> /I2C_SCL
- R14 pad 2: Net-(R14-Pad2) -> +3V3
- R15 pad 1: +3V3 -> Net-(C8-Pad1)
- R15 pad 2: Net-(R15-Pad2) -> +3V3
- R16 pad 1: Net-(Q7-Pad2) -> /I2C_SDA
- R16 pad 2: /USB_EN_A -> +3V3
- U6 pad 1: Net-(R15-Pad2) -> GND
- U6 pad 2: Net-(Q6-Pad3) -> /P2_LED_C
- U6 pad 3: Net-(J14-Pad1) -> /P3_LED_C
- U6 pad 4: Net-(J16-Pad1) -> /P3_LED_B
- U7 pad 11: unconnected-(U7-Pad11) -> /IR_BTN
- U7 pad 12: unconnected-(U7-Pad12) -> /LED_0
- U7 pad 13: unconnected-(U7-Pad13) -> /LED_1
- U7 pad 14: unconnected-(U7-Pad14) -> /I2C_SCL
- U7 pad 15: unconnected-(U7-Pad15) -> /I2C_SDA
- U7 pad 16: unconnected-(U7-Pad16) -> +3V3
- U7 pad 17: /IR_RLY_OUT -> GND
- U7 pad 18: /IR_RLY_IN -> GND
- U7 pad 19: /IR_BTN -> GND
- U7 pad 2: /RS232_RX -> /P2_SW_2
- U7 pad 20: /IR_LED -> +3V3
- U7 pad 21: /LED_0 -> /P4_SW_2
- U7 pad 22: /LED_1 -> /P4_SW_1
- U7 pad 23: /IO_0 -> /P4_SW_0
- U7 pad 24: /IO_1 -> /P3_SW_0
- U7 pad 25: /USB_EN_B -> /P3_SW_1
- U7 pad 26: /USB_EN_A -> /P3_SW_2
- U7 pad 27: /P3_LED_A -> /P2_SW_0
- U7 pad 28: /P3_LED_B -> /P2_SW_1
- U7 pad 3: /RS232_TX -> /P1_SW_2
- U7 pad 4: /P1_LED_A -> /P1_SW_1
- U7 pad 5: /P1_LED_B -> /P1_SW_0
- U7 pad 6: /P1_LED_C -> /INT
- U7 pad 7: /P1_SW_0 -> /IR_RLY_IN
- U7 pad 8: /P1_SW_1 -> GND
- U7 pad 9: /P1_SW_2 -> Net-(C7-Pad1)
- U8 pad 2: Net-(Q7-Pad3) -> unconnected-(U8-Pad2)
- U8 pad 3: Net-(J17-Pad1) -> GND
- U8 pad 4: Net-(J19-Pad1) -> unconnected-(U8-Pad4)
Routing:
- net +7.5V: track 0.00 -> 286.6 mm
- net +3V3: track 0.00 -> 279.7 mm, vias 0 -> 1
- net /P2_LED_C: track 0.00 -> 147.3 mm
- net +5V: track 4.73 -> 151.3 mm, vias 0 -> 1
- net /P2_SW_0: track 0.00 -> 133.8 mm
- net /P2_LED_B: track 0.00 -> 133.1 mm
- net /P2_LED_A: track 0.00 -> 126.9 mm
- net Net-(Q4-Pad2): track 0.00 -> 126.6 mm
- net /P2_SW_1: track 0.00 -> 122.9 mm
- net Net-(Q3-Pad3): track 0.00 -> 119.6 mm
- net +12V: track 90.7 -> 210.2 mm
- net Net-(Q1-Pad2): track 0.00 -> 111.7 mm
- net /P2_SW_2: track 0.00 -> 105.1 mm
- net /P1_LED_C: track 0.00 -> 104.7 mm
- net /P1_LED_B: track 0.00 -> 104.0 mm
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- added copper zone on B.Cu, net GND
- added copper zone on F.Cu, net GND
Other:
- board text added: "!"
- board text added: "+12V DC Power"
- board text added: "ADC Theatre SM Desk Video Switcher v1 - John Evans 2022 github.com/jevans3142/sm-desk-video-control"
- board text added: "Annunciators: LED0+ LED0- LED1+ LED1-"
- board text added: "Aux connector: +12V IO0 +5V IO1 GND"
- board text added: "IR Button:"
- board text added: "IR Relay Alt PSU link ->"
- board text added: "IR: Relay Sense GND GND"
- board text added: "LED+ LED- Button Button"
- board text added: "Link uC to 5V rail DO NOT USE if PoE in use"
- board text added: "Micro SD Card underneath module ↓"
- board text added: "Panel 1"
- board text added: "Panel 2"
- board text added: "Panel 3"
- board text added: "Panel 4"
- board text added: "UNPLUG 12V POWER BEFORE CONNECTING USB!"
- board text added: "USB Enables: +3.3V GND EN_A EN_B"
